File: sparkie.kicad_pcb (KiCad board)
At the start: 2 copper layers, 97.1 x 67.9 mm, 73 parts, among them J10 MotorAL, J11 MotorAR, J12 SERVO_0, J13 SERVO_1, J14 DEBUG, J15 AIR_SENSOR, J16 RST_BTN, J17 SERIAL, J18 ActionBtn, J19 Power5V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

Commit message: Changed name to 'Sparkie'
Parts:
- moved H1 35.1 mm to (234.3, 83.8)
- moved C12 22.8 mm to (200.7, 92.1)
- moved C13 14.0 mm to (201.2, 106.7)
- moved R12 1.27 mm to (182.9, 88.3)
- moved R11 1.27 mm to (181.0, 88.3)
Connections:
- U1 pad 9: unconnected-(U1-AD0-Pad9) -> GND
Routing:
- net GND: track 162.7 -> 211.5 mm, vias 14 -> 15
- net +12V: track 67.4 -> 47.0 mm, vias 2 -> 0
- net /USB_D+: track 36.9 -> 32.7 mm, vias 2 -> 0
- net Net-(J22-CC1): track 11.3 -> 15.3 mm, vias 0 -> 2
- net /USB_D-: track 34.1 -> 30.9 mm, vias 2 -> 0
- net Net-(J22-CC2): track 11.9 -> 13.8 mm
- net /MotorA_ENC1: track 54.4 -> 56.0 mm
- net /MotorA_ENC0: track 46.8 -> 48.3 mm
- net Net-(U5-USB_DM): track 7.25 -> 6.72 mm
- net Net-(U5-USB_DP): track 7.23 -> 6.71 mm
Other:
- board text added: "Sparkie Board v1.0"
- board text removed: "Hubbie Board v1.0"
