File: sparkie.kicad_sch (KiCad schematic)
At the start: 73 parts, among them J10 MotorAL, J11 MotorAR, J12 SERVO_0, J13 SERVO_1, J14 DEBUG, J15 AIR_SENSOR, J16 RST_BTN, J17 SERIAL, J18 ActionBtn, J19 Power5V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

Commit message: Changed name to 'Sparkie'
Connections:
- net GND: now also U1.9 (AD0)
- no-connect marks 6 -> 5
Other:
- title: hubbie_mboard -> Sparkie Embedded Board
